Commit message: update (finished Gazebo)

File: my_robot_description/urdf/common_properties.xacro (robot description, xacro)
@@ -11,4 +11,10 @@
     <material name="gray">
         <color rgba="0.5 0.5 0.5 1.0"/>
+    </material>
+    <material name="orange">
+        <color rgba="1.0 0.4 0 1.0"/>
+    </material>
+    <material name="yellow">
+        <color rgba="1.0 1.0 0 1.0"/>
     </material>
     <xacro:macro name="box_inertia" params="m x y z o_xyz o_rpy">

File: my_robot_description/urdf/my_robot.urdf.xacro (robot description, xacro)
@@ -4,4 +4,11 @@
     <xacro:include filename="mobile_base.xacro" />
     <xacro:include filename="mobile_base_gazebo.xacro" />
-    <xacro:include filename="camera.xacro" />
+    <xacro:include filename="arm.xacro" />
+    <xacro:include filename="arm_gazebo.xacro" />
+    <!-- <xacro:include filename="camera.xacro" /> -->
+    <joint name="mobile_base_arm_joint" type="fixed">
+        <parent link="base_link"/>
+        <child link="arm_base_link"/>
+        <origin xyz="${base_length/4.0} 0 ${base_height}" rpy="0 0 0"/>
+    </joint>
 </robot>
