Commit message: update (till ros_control 2-8)

File: my_robot_description/urdf/my_robot.urdf.xacro (robot description, xacro)
@@ -3,12 +3,13 @@
     <xacro:include filename="common_properties.xacro" />
     <xacro:include filename="mobile_base.xacro" />
-    <xacro:include filename="mobile_base_gazebo.xacro" />
-    <xacro:include filename="arm.xacro" />
-    <xacro:include filename="arm_gazebo.xacro" />
+    <xacro:include filename="mobile_base.ros2_control.xacro" />
+    <!-- <xacro:include filename="mobile_base_gazebo.xacro" /> -->
+    <!-- <xacro:include filename="arm.xacro" />
+    <xacro:include filename="arm_gazebo.xacro" /> -->
     <!-- <xacro:include filename="camera.xacro" /> -->
-    <joint name="mobile_base_arm_joint" type="fixed">
+    <!-- <joint name="mobile_base_arm_joint" type="fixed">
         <parent link="base_link"/>
         <child link="arm_base_link"/>
         <origin xyz="${base_length/4.0} 0 ${base_height}" rpy="0 0 0"/>
-    </joint>
+    </joint> -->
 </robot>
